File: hardware/KiCAD_Project/Open_Field_Logger_Lab.kicad_sch (KiCad schematic)
At the start: 61 parts, among them J1 1-0001899, J10 1-0001894, J11 1-0000127, J12 NP_Conn_01x06, J13 NP_Conn_01x03, J14 AUX Input, J2 1-0001899, J3 1-0001899, J4 1-0001899, J5 1-0001899, J6 1-0001899, J7 Conn_01x01, J8 NP_Conn_01x04, J9 1-0001894, Q1 1-0000163, Q2 1-0000163, Q3 1-0000163, SW1 1-0000681, U1 1-0001891, U2 1-0001892, U3 1-0001893, U4 1-0001890, Y1 1-0001901

Commit message: Rev 1.0 production files
Parts:
- renumbered C5 to C1, C16 to C5, C1 to C6, D3 to D1, D4 to D3, D1 to D4, H4 to H1, H3 to H2, H2 to H3, H1 to H4, J6 to J10, J2 to J11, J3 to J12, J4 to J13, J5 to J14, J9 to J2, J10 to J3, J14 to J4, J13 to J5, J12 to J6, J8 to J7, J11 to J8, J7 to J9, Q2 to Q1, Q1 to Q2, R4 to R1, R12 to R10, R14 to R11, R20 to R12, R1 to R14, R8 to R15, R7 to R16, R6 to R17, R5 to R18, R3 to R2, R15 to R3, R2 to R4, R21 to R5, R9 to R6, R11 to R7, R24 to R8, R10 to R9, U3 to U1, U4 to U2, U2 to U3, U1 to U4

Commit message: Fixed Issues: #2 #3 #4
Parts:
- PCB1: Internal Part Number 3-0000304 -> 3-0000307
Changed lines of the file:
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@@
 	(title_block
 		(title "Open Field Logger Lab PCB")
-		(date "2026-06-11")
-		(rev "1.0")
+		(date "2026-06-29")
+		(rev "1.1")
 		(company "Leeman Geophysical LLC")
 		(comment 1 "(479) 373-3736")
@@
 			)
 		)
-		(property "Internal Part Number" "3-0000304"
+		(property "Internal Part Number" "3-0000307"
 			(at 17.78 168.91 0)
 			(effects

Commit message: Issue Revision: #6
Parts:
- BT1, D1, D3, J1, J10, J11, J12, J13, J14, J2, J3, MI1, TH1, U1, U2, U3: Populated 1 -> 0
Changed lines of the file:
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@@
 			)
 		)
-		(property "Populated" "1"
+		(property "Populated" "0"
 			(at 55.372 30.226 0)
 			(effects
@@
 			)
 		)
-		(property "Populated" "1"
+		(property "Populated" "0"
 			(at 71.12 31.75 0)
 			(effects
@@
 			)
 		)
-		(property "Populated" "1"
+		(property "Populated" "0"
 			(at 232.41 116.84 0)
 			(effects
@@
 			)
 		)
-		(property "Populated" "1"
+		(property "Populated" "0"
 			(at 232.41 93.98 0)
 			(effects
@@
 			)
 		)
-		(property "Populated" "1"
+		(property "Populated" "0"
 			(at 68.58 135.89 0)
 			(effects
@@
 			)
 		)
-		(property "Populated" "1"
+		(property "Populated" "0"
 			(at 232.41 109.22 0)
 			(effects
@@
 			)
 		)
-		(property "Populated" "1"
+		(property "Populated" "0"
 			(at 232.41 101.6 0)
 			(effects
@@
 			)
 		)
-		(property "Populated" "1"
+		(property "Populated" "0"
 			(at 73.914 130.048 0)
 			(effects
@@
 			)
 		)
-		(property "Populated" "1"
+		(property "Populated" "0"
 			(at 232.41 124.46 0)
 			(effects
@@
 			)
 		)
-		(property "Populated" "1"
+		(property "Populated" "0"
 			(at 44.45 38.1 0)
 			(effects
@@
 			)
 		)
-		(property "Populated" "1"
+		(property "Populated" "0"
 			(at 74.93 52.578 0)
 			(effects
@@
 			)
 		)
-		(property "Populated" "1"
+		(property "Populated" "0"
 			(at 39.37 22.86 0)
 			(effects
@@
 			)
 		)
-		(property "Populated" "1"
+		(property "Populated" "0"
 			(at 33.02 184.15 0)
 			(effects
@@
 			)
 		)
-		(property "Populated" "1"
+		(property "Populated" "0"
 			(at 29.21 31.75 0)
 			(effects
@@
 			)
 		)
-		(property "Populated" "1"
+		(property "Populated" "0"
 			(at 226.06 154.94 0)
 			(effects
@@
 			)
 		)
-		(property "Populated" "1"
+		(property "Populated" "0"
 			(at 41.91 26.67 0)
 			(effects
